File: Controls-LightingPCB_TestBoard.kicad_sch (KiCad schematic)
At the start: 52 parts, among them J1 +12V, J10 REGEN_SW, J11 CRUZ_ST_INDICATOR_33v, J12 CRUZ_EN_INDICATOR_33v, J13 REGEN_INDICATOR_33v, J14 NEU_INDICATOR_33v, J15 FOR_INDICATOR_33v, J16 REV_INDICATOR_33v, J17 EXTERNAL_RIGHTBLINK, J18 EXTERNAL_LEFTBLINK, J19 INTERNAL_RIGHTBLINK, J2 GND, J20 INTERNAL_LEFTBLINK, J21 EXTERNAL_HDLT, J22 EXTERNAL_BRAKELIGHT, J3 POWER_MINION, J4 POWER_LEADERBOARD, J5 TURN_SIGNAL_SW, J6 CRUISE_ENABLE, J7 CRUISE_SET, J8 HZD_SW, J9 F/R_SW, SW1 SW_SP3T, SW2 SW_SPST, SW3 SW_SPST, SW4 SW_SPST, SW5 SW_SP3T, SW6 SW_SPST

Commit message: board update
Parts:
- removed SW1, SW5: SW_SP3T, symbol Switch:SW_SP3T
- added U1, U2: SP3T, UTSVT_Special:M2024SS1W03BC, symbol utsvt-misc:SP3T
- J10, J11, J12, J13, J14, J15, J16, J17, J18, J19, J20, J21, J22, J3, J4, J6, J7, J8: footprint Connector_Molex:Molex_Micro-Fit_3.0_43650-0200_1x02_P3.00mm_Horizontal -> Connector_Molex:Molex_Micro-Fit_3.0_43650-0215_1x02_P3.00mm_Vertical
- J5, J9: footprint Connector_Molex:Molex_Micro-Fit_3.0_43650-0400_1x04_P3.00mm_Horizontal -> Connector_Molex:Molex_Micro-Fit_3.0_43650-0415_1x04_P3.00mm_Vertical
- R1, R2, R3, R4, R5, R6: value R -> 330
- R10, R11, R12, R7, R8, R9: value R -> 4.7k
- SW2, SW3, SW4, SW6: footprint (none) -> UTSVT_Special:2MS6T1B3M2QES
Connections:
- net at J9.1 (Pin_1): now also U2.1 (Out)
- net at J9.2 (Pin_2): now also U2.4 (Out)
- net at J9.3 (Pin_3): now also U2.2 (In)
- net at J9.4 (Pin_4): now also U2.6 (Out)
- net at J5.1 (Pin_1): now also U1.1 (Out)
- net at J5.2 (Pin_2): now also U1.4 (Out)
- net at J5.4 (Pin_4): now also U1.6 (Out)
- net at J5.3 (Pin_3): now also U1.2 (In)
- new net: U2.3 (Short), U2.5 (Short)
- new net: U1.3 (Short), U1.5 (Short)
Other:
- note added: "LEDS (3.3V)"
- note removed: "SWITCH LEDS (3.3V)"

Commit message: update QUAC
Parts:
- added H1, H2, H3, H4: MountingHole, MountingHole:MountingHole_3mm, symbol Mechanical:MountingHole
- added LOGO1: Logo_Placeholder, UTSVT_Special:UTSVT_Logo_Symbol, symbol utsvt-misc:Logo_Placeholder
- added LOGO2: Logo_Placeholder, UTSVT_Special:Hallock_Image_Tiny, symbol utsvt-misc:Logo_Placeholder
- D1: value CRUZ_ST_INDICATOR -> CRUZ ST IND
- D10, J20: value INTERNAL_LEFTBLINK -> INT LBLINK
- D11: value EXTERNAL_HDLT -> EXT HDLT
- D12: value EXTERNAL_BRAKELIGHT -> EXT BRAKE
- D2: value CRUZ_EN_INDICATOR -> CRUZ EN IND
- D3: value REGEN_INDICATOR -> REGEN IND
- D4: value NEU_INDICATOR -> NEU IND
- D5: value FOR_INDICATOR -> FOR IND
- D6: value REV_INDICATOR -> REV IND
- D7: value EXTERNAL_RIGHTBLINK -> EXT RBLINK
- D8: value EXTERNAL_LEFTBLINK -> EXT LBLINK
- D9, J19: value INTERNAL_RIGHTBLINK -> INT RBLINK
- J10: value REGEN_SW -> REGEN SW
- J11: value CRUZ_ST_INDICATOR_33v -> CRUZ ST IND
- J12: value CRUZ_EN_INDICATOR_33v -> CRUZ EN IND
- J13: value REGEN_INDICATOR_33v -> REGEN IND; footprint Connector_Molex:Molex_Micro-Fit_3.0_43650-0215_1x02_P3.00mm_Vertical -> Connector_Molex:Molex_Micro-Fit_3.0_43650-0200_1x02_P3.00mm_Horizontal
- J14: value NEU_INDICATOR_33v -> NEU IND; footprint Connector_Molex:Molex_Micro-Fit_3.0_43650-0215_1x02_P3.00mm_Vertical -> Connector_Molex:Molex_Micro-Fit_3.0_43650-0200_1x02_P3.00mm_Horizontal
- J15: value FOR_INDICATOR_33v -> FOR IND
- J16: value REV_INDICATOR_33v -> REV IND; footprint Connector_Molex:Molex_Micro-Fit_3.0_43650-0215_1x02_P3.00mm_Vertical -> Connector_Molex:Molex_Micro-Fit_3.0_43650-0200_1x02_P3.00mm_Horizontal
- J17: value EXTERNAL_RIGHTBLINK -> EXT RBLINK; footprint Connector_Molex:Molex_Micro-Fit_3.0_43650-0215_1x02_P3.00mm_Vertical -> Connector_Molex:Molex_Micro-Fit_3.0_43650-0200_1x02_P3.00mm_Horizontal
- J18: value EXTERNAL_LEFTBLINK -> EXT LBLINK; footprint Connector_Molex:Molex_Micro-Fit_3.0_43650-0215_1x02_P3.00mm_Vertical -> Connector_Molex:Molex_Micro-Fit_3.0_43650-0200_1x02_P3.00mm_Horizontal
- J21: value EXTERNAL_HDLT -> EXT HDLT; footprint Connector_Molex:Molex_Micro-Fit_3.0_43650-0215_1x02_P3.00mm_Vertical -> Connector_Molex:Molex_Micro-Fit_3.0_43650-0200_1x02_P3.00mm_Horizontal
- J22: value EXTERNAL_BRAKELIGHT -> EXT BRAKE; footprint Connector_Molex:Molex_Micro-Fit_3.0_43650-0215_1x02_P3.00mm_Vertical -> Connector_Molex:Molex_Micro-Fit_3.0_43650-0200_1x02_P3.00mm_Horizontal
- J3: value POWER_MINION -> POWER MINION
- J4: value POWER_LEADERBOARD -> POWER LEADER
- J5: value TURN_SIGNAL_SW -> TURN SIG SW
- J6: value CRUISE_ENABLE -> CRUISE EN; footprint Connector_Molex:Molex_Micro-Fit_3.0_43650-0215_1x02_P3.00mm_Vertical -> Connector_Molex:Molex_Micro-Fit_3.0_43650-0200_1x02_P3.00mm_Horizontal
- J7: value CRUISE_SET -> CRUISE SET; footprint Connector_Molex:Molex_Micro-Fit_3.0_43650-0215_1x02_P3.00mm_Vertical -> Connector_Molex:Molex_Micro-Fit_3.0_43650-0200_1x02_P3.00mm_Horizontal
- J8: value HZD_SW -> HZD SW; footprint Connector_Molex:Molex_Micro-Fit_3.0_43650-0215_1x02_P3.00mm_Vertical -> Connector_Molex:Molex_Micro-Fit_3.0_43650-0200_1x02_P3.00mm_Horizontal
- J9: value F/R_SW -> F/R SW
Other:
- note added: "0.1"
- note added: "Controls Minion Test PCB"
- moved on the sheet: D1, D10, D11, D12, D2, D3, D4, D5, D6, D7, D8, D9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
